Commit message: Established foundations on which to develop Navigation node

File: ros_bbauv2012/Logic/navigation_2D/description/bbauv2012.urdf (robot description, URDF)
Before this commit: robot Bumblebee, 2 links, 1 joints
Links:
- link base_link: geometry visual mesh filename=package://navigation_2D/description/bbauv2012.stl scale=0.001 0.001 0.001

Commit message: Merge.

File: ros_bbauv2012/Logic/navigation_2D/description/bbauv2012.urdf (robot description, URDF)
Before this commit: robot Bumblebee, 2 links, 1 joints
Links:
- removed link base_link
- link base_footprint: mass 0.0001 -> None; geometry visual box size=0.001 0.001 0.001
Joints:
- removed joint base_footprint_joint
